Commit message: upgrade_model and tf

File: urdf/urdf/Cyberdog_new_version.xacro (robot description, xacro)
@@ -6,7 +6,7 @@
 <link name="base_link">
   <inertial>
-    <origin xyz="-0.006085364526447137 -0.0013192736274497407 0.3912794723646684" rpy="0 0 0"/>
-    <mass value="79.901474415363"/>
-    <inertia ixx="0.481497" iyy="1.948657" izz="2.158894" ixy="-0.000887" iyz="-0.000127" ixz="-0.078451"/>
+    <origin xyz="0.008091068495439373 0.006531996239142384 0.353123699225949" rpy="0 0 0"/>
+    <mass value="79.89988947207421"/>
+    <inertia ixx="0.481483" iyy="1.948653" izz="2.158879" ixy="-0.000887" iyz="0.000127" ixz="0.078451"/>
   </inertial>
   <visual>
@@ -24,415 +24,415 @@
   </collision>
 </link>
-<link name="foot2_br_1">
-  <inertial>
-    <origin xyz="0.07006520870174893 1.4227437647451602e-07 -0.09502063578021544" rpy="0 0 0"/>
-    <mass value="0.7095711315921492"/>
-    <inertia ixx="0.002276" iyy="0.003811" izz="0.001577" ixy="0.0" iyz="-0.0" ixz="0.001844"/>
-  </inertial>
-  <visual>
-    <origin xyz="0.501914 -0.148086 -0.251186" rpy="0 0 0"/>
-    <geometry>
-      <mesh filename="package://Cyberdog_new_version_description/meshes/foot2_br_1.stl" scale="0.001 0.001 0.001"/>
-    </geometry>
-    <material name="silver"/>
-  </visual>
-  <collision>
-    <origin xyz="0.501914 -0.148086 -0.251186" rpy="0 0 0"/>
-    <geometry>
-      <mesh filename="package://Cyberdog_new_version_description/meshes/foot2_br_1.stl" scale="0.001 0.001 0.001"/>
-    </geometry>
-  </collision>
-</link>
-<link name="foot1_fl_1">
-  <inertial>
-    <origin xyz="0.07006522133920257 1.377833254434524e-07 -0.09501970080479138" rpy="0 0 0"/>
-    <mass value="0.7095720022612411"/>
-    <inertia ixx="0.002277" iyy="0.003812" izz="0.001577" ixy="0.0" iyz="-0.0" ixz="0.001844"/>
-  </inertial>
-  <visual>
-    <origin xyz="-0.008786 -0.148086 -0.251186" rpy="0 0 0"/>
-    <geometry>
-      <mesh filename="package://Cyberdog_new_version_description/meshes/foot1_fl_1.stl" scale="0.001 0.001 0.001"/>
-    </geometry>
-    <material name="silver"/>
-  </visual>
-  <collision>
-    <origin xyz="-0.008786 -0.148086 -0.251186" rpy="0 0 0"/>
-    <geometry>
-      <mesh filename="package://Cyberdog_new_version_description/meshes/foot1_fl_1.stl" scale="0.001 0.001 0.001"/>
-    </geometry>
-  </collision>
-</link>
-<link name="foot2_br_2">
-  <inertial>
-    <origin xyz="0.07006520870131377 -4.153793341232781e-07 -0.09502063578021547" rpy="0 0 0"/>
-    <mass value="0.7095711315921492"/>
-    <inertia ixx="0.002276" iyy="0.003811" izz="0.001577" ixy="0.0" iyz="-0.0" ixz="0.001844"/>
-  </inertial>
-  <visual>
-    <origin xyz="0.501914 0.150849 -0.251186" rpy="0 0 0"/>
-    <geometry>
-      <mesh filename="package://Cyberdog_new_version_description/meshes/foot2_br_2.stl" scale="0.001 0.001 0.001"/>
-    </geometry>
-    <material name="silver"/>
-  </visual>
-  <collision>
-    <origin xyz="0.501914 0.150849 -0.251186" rpy="0 0 0"/>
-    <geometry>
-      <mesh filename="package://Cyberdog_new_version_description/meshes/foot2_br_2.stl" scale="0.001 0.001 0.001"/>
-    </geometry>
-  </collision>
-</link>
-<link name="foot1_fr_1">
-  <inertial>
-    <origin xyz="0.07006516238741908 -4.161127108714968e-07 -0.09502103314351346" rpy="0 0 0"/>
-    <mass value="0.7095709358424983"/>
-    <inertia ixx="0.002276" iyy="0.003811" izz="0.001577" ixy="0.0" iyz="-0.0" ixz="0.001844"/>
-  </inertial>
-  <visual>
-    <origin xyz="-0.008786 0.150849 -0.251186" rpy="0 0 0"/>
-    <geometry>
-      <mesh filename="package://Cyberdog_new_version_description/meshes/foot1_fr_1.stl" scale="0.001 0.001 0.001"/>
-    </geometry>
-    <material name="silver"/>
-  </visual>
-  <collision>
-    <origin xyz="-0.008786 0.150849 -0.251186" rpy="0 0 0"/>
-    <geometry>
-      <mesh filename="package://Cyberdog_new_version_description/meshes/foot1_fr_1.stl" scale="0.001 0.001 0.001"/>
-    </geometry>
-  </collision>
-</link>
-<link name="leg1_bl_1">
-  <inertial>
-    <origin xyz="-0.04327621629023265 0.02026500137913348 -0.02575619420770553" rpy="0 0 0"/>
-    <mass value="5.623670463448883"/>
-    <inertia ixx="0.009701" iyy="0.026697" izz="0.0184" ixy="-9e-06" iyz="-1.1e-05" ixz="-0.008656"/>
-  </inertial>
-  <visual>
-    <origin xyz="0.315442 -0.128086 -0.382754" rpy="0 0 0"/>
-    <geometry>
-      <mesh filename="package://Cyberdog_new_version_description/meshes/leg1_bl_1.stl" scale="0.001 0.001 0.001"/>
-    </geometry>
-    <material name="silver"/>
-  </visual>
-  <collision>
-    <origin xyz="0.315442 -0.128086 -0.382754" rpy="0 0 0"/>
-    <geometry>
-      <mesh filename="package://Cyberdog_new_version_description/meshes/leg1_bl_1.stl" scale="0.001 0.001 0.001"/>
-    </geometry>
-  </collision>
-</link>
-<link name="bol2_r_1">
-  <inertial>
-    <origin xyz="3.3243352715039975e-07 -4.2306274966597e-07 -0.009973935277613359" rpy="0 0 0"/>
-    <mass value="0.15181620834766513"/>
-    <inertia ixx="1.7e-05" iyy="1.7e-05" izz="2.1e-05" ixy="-0.0" iyz="-0.0" ixz="0.0"/>
-  </inertial>
-  <visual>
-    <origin xyz="0.345101 0.150849 -0.063164" rpy="0 0 0"/>
-    <geometry>
-      <mesh filename="package://Cyberdog_new_version_description/meshes/bol2_r_1.stl" scale="0.001 0.001 0.001"/>
-    </geometry>
-    <material name="silver"/>
-  </visual>
-  <collision>
-    <origin xyz="0.345101 0.150849 -0.063164" rpy="0 0 0"/>
-    <geometry>
-      <mesh filename="package://Cyberdog_new_version_description/meshes/bol2_r_1.stl" scale="0.001 0.001 0.001"/>
-    </geometry>
-  </collision>
-</link>
-<link name="bol2_l__1">
-  <inertial>
-    <origin xyz="3.3243396413418225e-07 1.3459096870338527e-07 -0.009973935277615933" rpy="0 0 0"/>
-    <mass value="0.1518162083476651"/>
-    <inertia ixx="1.7e-05" iyy="1.7e-05" izz="2.1e-05" ixy="-0.0" iyz="-0.0" ixz="0.0"/>
-  </inertial>
-  <visual>
-    <origin xyz="0.345101 -0.148086 -0.063164" rpy="0 0 0"/>
-    <geometry>
-      <mesh filename="package://Cyberdog_new_version_description/meshes/bol2_l__1.stl" scale="0.001 0.001 0.001"/>
-    </geometry>
-    <material name="silver"/>
-  </visual>
-  <collision>
-    <origin xyz="0.345101 -0.148086 -0.063164" rpy="0 0 0"/>
-    <geometry>
-      <mesh filename="package://Cyberdog_new_version_description/meshes/bol2_l__1.stl" scale="0.001 0.001 0.001"/>
-    </geometry>
-  </collision>
-</link>
-<link name="bol1_r_1">
-  <inertial>
-    <origin xyz="3.327502144656602e-07 -4.2314786530273096e-07 -0.009973935982052443" rpy="0 0 0"/>
-    <mass value="0.1518162083476651"/>
-    <inertia ixx="1.7e-05" iyy="1.7e-05" izz="2.1e-05" ixy="-0.0" iyz="-0.0" ixz="0.0"/>
-  </inertial>
-  <visual>
-    <origin xyz="-0.165599 0.150849 -0.063164" rpy="0 0 0"/>
-    <geometry>
-      <mesh filename="package://Cyberdog_new_version_description/meshes/bol1_r_1.stl" scale="0.001 0.001 0.001"/>
-    </geometry>
-    <material name="silver"/>
-  </visual>
-  <collision>
-    <origin xyz="-0.165599 0.150849 -0.063164" rpy="0 0 0"/>
-    <geometry>
-      <mesh filename="package://Cyberdog_new_version_description/meshes/bol1_r_1.stl" scale="0.001 0.001 0.001"/>
-    </geometry>
-  </collision>
-</link>
-<link name="bol1_l_1">
-  <inertial>
-    <origin xyz="3.3275562749679466e-07 1.3450366534439873e-07 -0.009973935982524516" rpy="0 0 0"/>
-    <mass value="0.15181620834766513"/>
-    <inertia ixx="1.7e-05" iyy="1.7e-05" izz="2.1e-05" ixy="-0.0" iyz="-0.0" ixz="0.0"/>
-  </inertial>
-  <visual>
-    <origin xyz="-0.165599 -0.148086 -0.063164" rpy="0 0 0"/>
-    <geometry>
-      <mesh filename="package://Cyberdog_new_version_description/meshes/bol1_l_1.stl" scale="0.001 0.001 0.001"/>
-    </geometry>
-    <material name="silver"/>
-  </visual>
-  <collision>
-    <origin xyz="-0.165599 -0.148086 -0.063164" rpy="0 0 0"/>
-    <geometry>
-      <mesh filename="package://Cyberdog_new_version_description/meshes/bol1_l_1.stl" scale="0.001 0.001 0.001"/>
-    </geometry>
-  </collision>
-</link>
-<link name="leg1_fr_1">
-  <inertial>
-    <origin xyz="-0.04327621637241477 -0.019735556367151214 -0.025756194021132106" rpy="0 0 0"/>
-    <mass value="5.623670463448882"/>
-    <inertia ixx="0.009701" iyy="0.026697" izz="0.0184" ixy="-9e-06" iyz="-1.1e-05" ixz="-0.008656"/>
-  </inertial>
-  <visual>
-    <origin xyz="-0.195258 0.130849 -0.382754" rpy="0 0 0"/>
-    <geometry>
-      <mesh filename="package://Cyberdog_new_version_description/meshes/leg1_fr_1.stl" scale="0.001 0.001 0.001"/>
-    </geometry>
-    <material name="silver"/>
-  </visual>
-  <collision>
-    <origin xyz="-0.195258 0.130849 -0.382754" rpy="0 0 0"/>
-    <geometry>
-      <mesh filename="package://Cyberdog_new_version_description/meshes/leg1_fr_1.stl" scale="0.001 0.001 0.001"/>
-    </geometry>
-  </collision>
-</link>
-<link name="leg1_fl_1">
-  <inertial>
-    <origin xyz="-0.04327621636698725 0.020265001285029977 -0.025756194021603285" rpy="0 0 0"/>
-    <mass value="5.62367046344888"/>
-    <inertia ixx="0.009701" iyy="0.026697" izz="0.0184" ixy="-9e-06" iyz="-1.1e-05" ixz="-0.008656"/>
-  </inertial>
-  <visual>
-    <origin xyz="-0.195258 -0.128086 -0.382754" rpy="0 0 0"/>
-    <geometry>
-      <mesh filename="package://Cyberdog_new_version_description/meshes/leg1_fl_1.stl" scale="0.001 0.001 0.001"/>
-    </geometry>
-    <material name="silver"/>
-  </visual>
-  <collision>
-    <origin xyz="-0.195258 -0.128086 -0.382754" rpy="0 0 0"/>
-    <geometry>
-      <mesh filename="package://Cyberdog_new_version_description/meshes/leg1_fl_1.stl" scale="0.001 0.001 0.001"/>
-    </geometry>
-  </collision>
-</link>
-<link name="leg1_br_1">
-  <inertial>
-    <origin xyz="-0.0432762162906693 -0.019735556274586313 -0.025756194207707694" rpy="0 0 0"/>
-    <mass value="5.623670463448881"/>
-    <inertia ixx="0.009701" iyy="0.026697" izz="0.0184" ixy="-9e-06" iyz="-1.1e-05" ixz="-0.008656"/>
-  </inertial>
-  <visual>
-    <origin xyz="0.315442 0.130849 -0.382754" rpy="0 0 0"/>
-    <geometry>
-      <mesh filename="package://Cyberdog_new_version_description/meshes/leg1_br_1.stl" scale="0.001 0.001 0.001"/>
-    </geometry>
-    <material name="silver"/>
-  </visual>
-  <collision>
-    <origin xyz="0.315442 0.130849 -0.382754" rpy="0 0 0"/>
-    <geometry>
-      <mesh filename="package://Cyberdog_new_version_description/meshes/leg1_br_1.stl" scale="0.001 0.001 0.001"/>
-    </geometry>
-  </collision>
-</link>
-<link name="motor2_bl_back_1">
-  <inertial>
-    <origin xyz="-0.0696654751135935 0.025196011025119112 1.2772211338551998e-07" rpy="0 0 0"/>
-    <mass value="3.9545724305182866"/>
-    <inertia ixx="0.005455" iyy="0.00436" izz="0.006263" ixy="0.000503" iyz="0.0" ixz="-0.0"/>
-  </inertial>
-  <visual>
-    <origin xyz="0.240942 -0.050586 -0.382754" rpy="0 0 0"/>
-    <geometry>
-      <mesh filename="package://Cyberdog_new_version_description/meshes/motor2_bl_back_1.stl" scale="0.001 0.001 0.001"/>
-    </geometry>
-    <material name="silver"/>
-  </visual>
-  <collision>
-    <origin xyz="0.240942 -0.050586 -0.382754" rpy="0 0 0"/>
-    <geometry>
-      <mesh filename="package://Cyberdog_new_version_description/meshes/motor2_bl_back_1.stl" scale="0.001 0.001 0.001"/>
-    </geometry>
-  </collision>
-</link>
-<link name="motor1_br_back__1">
-  <inertial>
-    <origin xyz="-0.06966547511381554 -0.02519630009305559 1.2772211382960919e-07" rpy="0 0 0"/>
-    <mass value="3.954572430518811"/>
-    <inertia ixx="0.005455" iyy="0.00436" izz="0.006263" ixy="-0.000503" iyz="-0.0" ixz="-0.0"/>
-  </inertial>
-  <visual>
-    <origin xyz="0.240942 0.053349 -0.382754" rpy="0 0 0"/>
-    <geometry>
-      <mesh filename="package://Cyberdog_new_version_description/meshes/motor1_br_back__1.stl" scale="0.001 0.001 0.001"/>
-    </geometry>
-    <material name="silver"/>
-  </visual>
-  <collision>
-    <origin xyz="0.240942 0.053349 -0.382754" rpy="0 0 0"/>
-    <geometry>
-      <mesh filename="package://Cyberdog_new_version_description/meshes/motor1_br_back__1.stl" scale="0.001 0.001 0.001"/>
-    </geometry>
-  </collision>
-</link>
-<link name="motor1_br_1">
-  <inertial>
-    <origin xyz="0.07105512711142814 -0.025162590366412517 8.499528188488092e-07" rpy="0 0 0"/>
-    <mass value="3.9597418606976182"/>
-    <inertia ixx="0.005468" iyy="0.004405" izz="0.00631" ixy="0.000514" iyz="-0.0" ixz="-0.0"/>
-  </inertial>
-  <visual>
-    <origin xyz="-0.119258 0.053349 -0.382754" rpy="0 0 0"/>
-    <geometry>
-      <mesh filename="package://Cyberdog_new_version_description/meshes/motor1_br_1.stl" scale="0.001 0.001 0.001"/>
-    </geometry>
-    <material name="silver"/>
-  </visual>
-  <collision>
-    <origin xyz="-0.119258 0.053349 -0.382754" rpy="0 0 0"/>
-    <geometry>
-      <mesh filename="package://Cyberdog_new_version_description/meshes/motor1_br_1.stl" scale="0.001 0.001 0.001"/>
-    </geometry>
-  </collision>
-</link>
-<link name="motor1_bl_1">
-  <inertial>
-    <origin xyz="0.07105512711326073 0.025162301108794964 8.499524354887988e-07" rpy="0 0 0"/>
-    <mass value="3.9597418607827"/>
-    <inertia ixx="0.005468" iyy="0.004405" izz="0.00631" ixy="-0.000514" iyz="0.0" ixz="-0.0"/>
-  </inertial>
-  <visual>
-    <origin xyz="-0.119258 -0.050586 -0.382754" rpy="0 0 0"/>
-    <geometry>
-      <mesh filename="package://Cyberdog_new_version_description/meshes/motor1_bl_1.stl" scale="0.001 0.001 0.001"/>
-    </geometry>
-    <material name="silver"/>
-  </visual>
-  <collision>
-    <origin xyz="-0.119258 -0.050586 -0.382754" rpy="0 0 0"/>
-    <geometry>
-      <mesh filename="package://Cyberdog_new_version_description/meshes/motor1_bl_1.stl" scale="0.001 0.001 0.001"/>
-    </geometry>
-  </collision>
-</link>
-<joint name="Revolute 5" type="continuous">
-  <origin xyz="-0.186472 0.02 -0.131568" rpy="0 0 0"/>
-  <parent link="leg1_bl_1"/>
-  <child link="foot2_br_1"/>
-  <axis xyz="-0.0 -1.0 -0.0"/>
-</joint>
-<joint name="Revolute 6" type="continuous">
-  <origin xyz="-0.186472 0.02 -0.131568" rpy="0 0 0"/>
-  <parent link="leg1_fl_1"/>
-  <child link="foot1_fl_1"/>
+<link name="motor1_1">
+  <inertial>
+    <origin xyz="-0.07105472379758557 -0.025162567226755556 2.2426371465433803e-07" rpy="0 0 0"/>
+    <mass value="3.9597418607827164"/>
+    <inertia ixx="0.005468" iyy="0.004405" izz="0.00631" ixy="-0.000514" iyz="-0.0" ixz="0.0"/>
+  </inertial>
+  <visual>
+    <origin xyz="0.117253 0.045373 -0.344599" rpy="0 0 0"/>
+    <geometry>
+      <mesh filename="package://Cyberdog_new_version_description/meshes/motor1_1.stl" scale="0.001 0.001 0.001"/>
+    </geometry>
+    <material name="silver"/>
+  </visual>
+  <collision>
+    <origin xyz="0.117253 0.045373 -0.344599" rpy="0 0 0"/>
+    <geometry>
+      <mesh filename="package://Cyberdog_new_version_description/meshes/motor1_1.stl" scale="0.001 0.001 0.001"/>
+    </geometry>
+  </collision>
+</link>
+<link name="foot1_1">
+  <inertial>
+    <origin xyz="7.055885262174932e-08 -4.006286399571568e-07 -0.009973561669559806" rpy="0 0 0"/>
+    <mass value="0.15181620834766546"/>
+    <inertia ixx="1.7e-05" iyy="1.7e-05" izz="2.1e-05" ixy="0.0" iyz="0.0" ixz="-0.0"/>
+  </inertial>
+  <visual>
+    <origin xyz="0.163594 0.142873 -0.025008" rpy="0 0 0"/>
+    <geometry>
+      <mesh filename="package://Cyberdog_new_version_description/meshes/foot1_1.stl" scale="0.001 0.001 0.001"/>
+    </geometry>
+    <material name="silver"/>
+  </visual>
+  <collision>
+    <origin xyz="0.163594 0.142873 -0.025008" rpy="0 0 0"/>
+    <geometry>
+      <mesh filename="package://Cyberdog_new_version_description/meshes/foot1_1.stl" scale="0.001 0.001 0.001"/>
+    </geometry>
+  </collision>
+</link>
+<link name="motor0_1">
+  <inertial>
+    <origin xyz="-0.07105472379596117 0.02516232424838287 2.2426031059952223e-07" rpy="0 0 0"/>
+    <mass value="3.9597418607117993"/>
+    <inertia ixx="0.005468" iyy="0.004405" izz="0.00631" ixy="0.000514" iyz="0.0" ixz="0.0"/>
+  </inertial>
+  <visual>
+    <origin xyz="0.117253 -0.058562 -0.344599" rpy="0 0 0"/>
+    <geometry>
+      <mesh filename="package://Cyberdog_new_version_description/meshes/motor0_1.stl" scale="0.001 0.001 0.001"/>
+    </geometry>
+    <material name="silver"/>
+  </visual>
+  <collision>
+    <origin xyz="0.117253 -0.058562 -0.344599" rpy="0 0 0"/>
+    <geometry>
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